Commit message: Made robot bigger and with added weight

File: urdf/robot.xacro (robot description, xacro)
@@ -10,10 +10,34 @@
     <origin xyz="0 0 0" rpy="0 0 0" />
     <parent link="robot_footprint"/>
-    <child link="chassis" />
-  </joint>
+    <child link="base_link" />
+  </joint>
+  <link name='base_link'>
+    <pose>0 0 0.1 0 0 0</pose>
+    <inertial>
+      <mass value="20.0"/>
+      <origin xyz="0.0 0 0" rpy=" 0 0 0"/>
+      <inertia
+          ixx="0.1" ixy="0" ixz="0"
+          iyy="0.1" iyz="0"
+          izz="0.1"
+      />
+    </inertial>
+    <collision name='collision'>
+      <origin xyz="0 0 0" rpy=" 0 0 0"/>
+      <geometry>
+        <box size=".5 .35 .08"/>
+      </geometry>
+    </collision>
+    <visual name='base_link_visual'>
+      <origin xyz="0 0 0" rpy=" 0 0 0"/>
+      <geometry>
+        <box size=".5 .35 .08"/>
+      </geometry>
+    </visual>
+  </link>
   <link name='chassis'>
     <pose>0 0 0.1 0 0 0</pose>
     <inertial>
-      <mass value="5.0"/>
+      <mass value="20.0"/>
       <origin xyz="0.0 0 0" rpy=" 0 0 0"/>
       <inertia
@@ -26,5 +50,5 @@
       <origin xyz="0 0 0" rpy=" 0 0 0"/>
       <geometry>
-        <box size=".4 .3 .08"/>
+        <box size=".4 .3 .30"/>
       </geometry>
     </collision>
@@ -32,8 +56,14 @@
       <origin xyz="0 0 0" rpy=" 0 0 0"/>
       <geometry>
-        <box size=".4 .3 .08"/>
-      </geometry>
-    </visual>
-  </link>
+        <box size=".4 .3 .30"/>
+      </geometry>
+    </visual>
+  </link>
+  <joint name="base_link_chassis_joint" type="fixed">
+    <axis xyz="0 1 0" />
+    <origin xyz="0 0 0.1" rpy="0 0 0"/>
+    <parent link="base_link"/>
+    <child link="chassis"/>
+  </joint>
   <link name='front_left_wheel'>
     <commandTopic>cmd_vel</commandTopic>
@@ -207,5 +237,5 @@
   <joint name="imu_joint" type="fixed">
     <axis xyz="0 1 0" />
-    <origin xyz="0 0 0.08" rpy="0 0 0"/>
+    <origin xyz="0 0 0.18" rpy="0 0 0"/>
     <parent link="chassis"/>
     <child link="imu"/>
@@ -213,12 +243,12 @@
   <joint name="gps_joint" type="fixed">
     <axis xyz="0 1 0" />
-    <origin xyz="-0.15 0 0.08" rpy="0 0 0"/>
+    <origin xyz="-0.15 0 0.18" rpy="0 0 0"/>
     <parent link="chassis"/>
     <child link="gps"/>
   </joint>
   <joint type="continuous" name="front_left_wheel_joint">
-    <origin xyz="0.15 0.18 0" rpy="0 0 0"/>
+    <origin xyz="0.15 0.22 0" rpy="0 0 0"/>
     <child link="front_left_wheel"/>
-    <parent link="chassis"/>
+    <parent link="base_link"/>
     <axis xyz="0 1 0" rpy="0 0 0"/>
     <limit effort="10000" velocity="1000"/>
@@ -226,7 +256,7 @@
   </joint>
   <joint type="continuous" name="front_right_wheel_joint">
-    <origin xyz="0.15 -0.18 0" rpy="0 0 0"/>
+    <origin xyz="0.15 -0.22 0" rpy="0 0 0"/>
     <child link="front_right_wheel"/>
-    <parent link="chassis"/>
+    <parent link="base_link"/>
     <axis xyz="0 1 0" rpy="0 0 0"/>
     <limit effort="10000" velocity="1000"/>
@@ -234,7 +264,7 @@
   </joint>
   <joint type="continuous" name="back_left_wheel_joint">
-    <origin xyz="-0.15 0.18 0" rpy="0 0 0"/>
+    <origin xyz="-0.15 0.22 0" rpy="0 0 0"/>
     <child link="back_left_wheel"/>
-    <parent link="chassis"/>
+    <parent link="base_link"/>
     <axis xyz="0 1 0" rpy="0 0 0"/>
     <limit effort="10000" velocity="1000"/>
@@ -242,7 +272,7 @@
   </joint>
   <joint type="continuous" name="back_right_wheel_joint">
-    <origin xyz="-0.15 -0.18 0" rpy="0 0 0"/>
+    <origin xyz="-0.15 -0.22 0" rpy="0 0 0"/>
     <child link="back_right_wheel"/>
-    <parent link="chassis"/>
+    <parent link="base_link"/>
     <axis xyz="0 1 0" rpy="0 0 0"/>
     <limit effort="10000" velocity="1000"/>
@@ -265,5 +295,5 @@
   <xacro:include filename="$(find robosense_description)/urdf/RS-16.urdf.xacro"/>
   <RS-16 parent="chassis" name="robosense" topic="/rslidar_points" hz="10" samples="900" gpu="${gpu}">
-    <origin xyz=".15 0 0.14" rpy="0 0 0" />
+    <origin xyz=".15 0 0.24" rpy="0 0 0" />
   </RS-16>
 </robot>

Commit message: Increased model weight and torque

File: urdf/robot.xacro (robot description, xacro)
@@ -15,5 +15,5 @@
     <pose>0 0 0.1 0 0 0</pose>
     <inertial>
-      <mass value="20.0"/>
+      <mass value="40.0"/>
       <origin xyz="0.0 0 0" rpy=" 0 0 0"/>
       <inertia

Commit message: Updated to publish tf and increased robot weight

File: urdf/robot.xacro (robot description, xacro)
@@ -15,5 +15,5 @@
     <pose>0 0 0.1 0 0 0</pose>
     <inertial>
-      <mass value="40.0"/>
+      <mass value="50.0"/>
       <origin xyz="0.0 0 0" rpy=" 0 0 0"/>
       <inertia
@@ -39,5 +39,5 @@
     <pose>0 0 0.1 0 0 0</pose>
     <inertial>
-      <mass value="20.0"/>
+      <mass value="30.0"/>
       <origin xyz="0.0 0 0" rpy=" 0 0 0"/>
       <inertia
@@ -294,5 +294,5 @@
   <xacro:property name="gpu" value="$(arg gpu)" />
   <xacro:include filename="$(find robosense_description)/urdf/RS-16.urdf.xacro"/>
-  <RS-16 parent="chassis" name="robosense" topic="/rslidar_points" hz="10" samples="200" gpu="${gpu}">
+  <RS-16 parent="chassis" name="robosense" topic="/rslidar_points" hz="10" samples="150" gpu="${gpu}">
     <origin xyz=".15 0 0.24" rpy="0 0 0" />
   </RS-16>

Commit message: Added sonar, reduced weight and updated visuals

File: urdf/robot.xacro (robot description, xacro)
@@ -15,5 +15,5 @@
     <pose>0 0 0.1 0 0 0</pose>
     <inertial>
-      <mass value="50.0"/>
+      <mass value="40.0"/>
       <origin xyz="0.0 0 0" rpy=" 0 0 0"/>
       <inertia
@@ -39,5 +39,5 @@
     <pose>0 0 0.1 0 0 0</pose>
     <inertial>
-      <mass value="30.0"/>
+      <mass value="20.0"/>
       <origin xyz="0.0 0 0" rpy=" 0 0 0"/>
       <inertia
@@ -66,4 +66,23 @@
     <child link="chassis"/>
   </joint>
+  <link name='neck'>
+    <collision name='collision'>
+      <origin xyz="0 0 0" rpy=" 0 0 0"/>
+      <geometry>
+        <cylinder length="0.55" radius="0.04"/>
+      </geometry>
+    </collision>
+    <visual name='chassis_visual'>
+      <origin xyz="0 0 0" rpy=" 0 0 0"/>
+      <geometry>
+        <cylinder length="0.55" radius="0.04"/>
+      </geometry>
+    </visual>
+  </link>
+  <joint name="chassis_neck_joint" type="fixed">
+    <origin xyz="0.15 0 0.3" rpy="0 0 0"/>
+    <parent link="chassis"/>
+    <child link="neck"/>
+  </joint>
   <link name='front_left_wheel'>
     <commandTopic>cmd_vel</commandTopic>
@@ -82,4 +101,14 @@
         <cylinder radius="0.12" length="0.04"/>
       </geometry>
+      <surface>
+      <contact>
+        <ode>
+   		<mu1 value="200.0"/>
+    		<mu2 value="100.0"/>
+    		<kp value="10000000.0" />
+    		<kd value="1.0" />
+        </ode>
+      </contact>
+      </surface>
     </collision>
     <visual name='visual'>
@@ -93,17 +122,27 @@
     <commandTopic>cmd_vel</commandTopic>
     <inertial>
-      <mass value="5.0"/>
-      <origin xyz="0 0 0" rpy="0 1.5707 1.5707"/>
-      <inertia
-          ixx="0.1" ixy="0" ixz="0"
-          iyy="0.1" iyz="0"
-          izz="0.1"
-      />
-    </inertial>
-    <collision name='collision'>
-      <origin xyz="0 0 0" rpy="0 1.5707 1.5707"/>
-      <geometry>
-        <cylinder radius="0.12" length="0.04"/>
-      </geometry>
+      <mass value="4.0"/>
+      <origin xyz="0 0 0" rpy="0 1.5707 1.5707"/>
+      <inertia
+          ixx="0.1" ixy="0" ixz="0"
+          iyy="0.1" iyz="0"
+          izz="0.1"
+      />
+    </inertial>
+    <collision name='collision'>
+      <origin xyz="0 0 0" rpy="0 1.5707 1.5707"/>
+      <geometry>
+        <cylinder radius="0.12" length="0.04"/>
+      </geometry>
+      <surface>
+      <contact>
+        <ode>
+   		<mu1 value="200.0"/>
+    		<mu2 value="100.0"/>
+    		<kp value="10000000.0" />
+    		<kd value="1.0" />
+        </ode>
+      </contact>
+      </surface>
     </collision>
     <visual name='visual'>
@@ -130,4 +169,14 @@
         <cylinder radius="0.12" length="0.04"/>
       </geometry>
+      <surface>
+      <contact>
+        <ode>
+   		<mu1 value="200.0"/>
+    		<mu2 value="100.0"/>
+    		<kp value="10000000.0" />
+    		<kd value="1.0" />
+        </ode>
+      </contact>
+      </surface>
     </collision>
     <visual name='visual'>
@@ -141,17 +190,27 @@
     <commandTopic>cmd_vel</commandTopic>
     <inertial>
-      <mass value="5.0"/>
-      <origin xyz="0 0 0" rpy="0 1.5707 1.5707"/>
-      <inertia
-          ixx="0.1" ixy="0" ixz="0"
-          iyy="0.1" iyz="0"
-          izz="0.1"
-      />
-    </inertial>
-    <collision name='collision'>
-      <origin xyz="0 0 0" rpy="0 1.5707 1.5707"/>
-      <geometry>
-        <cylinder radius="0.12" length="0.04"/>
-      </geometry>
+      <mass value="4.0"/>
+      <origin xyz="0 0 0" rpy="0 1.5707 1.5707"/>
+      <inertia
+          ixx="0.1" ixy="0" ixz="0"
+          iyy="0.1" iyz="0"
+          izz="0.1"
+      />
+    </inertial>
+    <collision name='collision'>
+      <origin xyz="0 0 0" rpy="0 1.5707 1.5707"/>
+      <geometry>
+        <cylinder radius="0.12" length="0.04"/>
+      </geometry>
+      <surface>
+      <contact>
+        <ode>
+   		<mu1 value="200.0"/>
+    		<mu2 value="100.0"/>
+    		<kp value="10000000.0" />
+    		<kd value="1.0" />
+        </ode>
+      </contact>
+      </surface>
     </collision>
     <visual name='visual'>
@@ -235,4 +294,54 @@
     </inertial>
   </link>
+  <link name="base_sonar_front">
+    <collision>
+      <origin xyz="0 0 0" rpy="0 0 0"/>
+      <geometry>
+        <box size="0.01 0.01 0.01"/>
+      </geometry>
+    </collision>    <visual>
+      <origin xyz="0 0 0" rpy="0 0 0"/>
+      <geometry>
+        <box size="0.01 0.01 0.01"/>
+      </geometry>
+      <material name="blue"/>
+    </visual>
+    <inertial>
+      <mass value="1e-5" />
+      <origin xyz="0 0 0" rpy="0 0 0"/>
+      <inertia ixx="1e-6" ixy="0" ixz="0" iyy="1e-6" iyz="0" izz="1e-6" />
+    </inertial>
+ </link>
+ <link name="base_sonar_rear">
+    <collision>
+      <origin xyz="0 0 0" rpy="0 0 0"/>
+      <geometry>
+        <box size="0.01 0.01 0.01"/>
+      </geometry>
+    </collision>    <visual>
+      <origin xyz="0 0 0" rpy="0 0 0"/>
+      <geometry>
+        <box size="0.01 0.01 0.01"/>
+      </geometry>
+      <material name="blue"/>
+    </visual>
+    <inertial>
+      <mass value="1e-5" />
+      <origin xyz="0 0 0" rpy="0 0 0"/>
+      <inertia ixx="1e-6" ixy="0" ixz="0" iyy="1e-6" iyz="0" izz="1e-6" />
+    </inertial>
+ </link>
+ <joint name="sonar_front_joint" type="fixed">
+    <axis xyz="0 1 0" />
+    <origin rpy="0 0 0" xyz="0.25 0 0.2" />
+    <parent link="base_link"/>
+    <child link="base_sonar_front"/>
+  </joint>
+  <joint name="sonar_front_rear" type="fixed">
+    <axis xyz="0 1 0" />
+    <origin rpy="0 0 3.14" xyz="-0.25 0 0.2" />
+    <parent link="base_link"/>
+    <child link="base_sonar_rear"/>
+  </joint>
   <joint name="imu_joint" type="fixed">
     <axis xyz="0 1 0" />
@@ -295,5 +404,5 @@
   <xacro:include filename="$(find robosense_description)/urdf/RS-16.urdf.xacro"/>
   <RS-16 parent="chassis" name="robosense" topic="/rslidar_points" hz="10" samples="150" gpu="${gpu}">
-    <origin xyz=".15 0 0.24" rpy="0 0 0" />
+    <origin xyz=".15 0 0.6" rpy="0 0 0" />
   </RS-16>
 </robot>

Commit message: added lidar->scan tf

File: urdf/robot.xacro (robot description, xacro)
@@ -338,5 +338,5 @@
     <child link="base_sonar_front"/>
   </joint>
-  <joint name="sonar_front_rear" type="fixed">
+  <joint name="sonar_rear_joint" type="fixed">
     <axis xyz="0 1 0" />
     <origin rpy="0 0 3.14" xyz="-0.25 0 0.2" />
@@ -403,6 +403,13 @@
   <xacro:property name="gpu" value="$(arg gpu)" />
   <xacro:include filename="$(find robosense_description)/urdf/RS-16.urdf.xacro"/>
-  <RS-16 parent="chassis" name="robosense" topic="/rslidar_points" hz="10" samples="150" gpu="${gpu}">
+  <RS-16 parent="chassis" name="rslidar" topic="/rslidar_points" hz="10" samples="150" gpu="${gpu}">
     <origin xyz=".15 0 0.6" rpy="0 0 0" />
   </RS-16>
+<link name='scan'/>
+ <joint type="fixed" name="link_lidar_scan_broadcaster">
+    <origin xyz="0 0 0" rpy="0 0 0"/>
+    <child link="scan"/>
+    <parent link="rslidar"/>
+    <axis xyz="0 0 0" rpy="0 0 0"/>
+  </joint>
 </robot>

Commit message: Updated footprint base_link joint

File: urdf/robot.xacro (robot description, xacro)
@@ -8,5 +8,5 @@
   <link name="robot_footprint"></link>
   <joint name="robot_footprint_joint" type="fixed">
-    <origin xyz="0 0 0" rpy="0 0 0" />
+    <origin xyz="0 0 0.05" rpy="0 0 0" />
     <parent link="robot_footprint"/>
     <child link="base_link" />

Commit message: added pan tilt model to chassis

File: urdf/robot.xacro (robot description, xacro)
@@ -2,4 +2,5 @@
 <robot name="robot" xmlns:xacro="http://www.ros.org/wiki/xacro">
   <xacro:include filename="$(find robot_model)/urdf/robot.gazebo" />
+  <xacro:include filename="$(find robot_model)/urdf/pan_tilt.xacro"/>
   <xacro:property name="imu_size" value="0.03"/>
   <xacro:property name="imu_mass" value="0.05"/>
@@ -221,5 +222,5 @@
     </visual>
   </link>
-  <link name='camera'>
+  <!-- <link name='camera'>
     <imageTopicName>rgb/image_raw</imageTopicName>
     <inertial>
@@ -251,5 +252,5 @@
     </visual>
   </link>
-  <link name="camera_link_optical"></link>
+  <link name="camera_link_optical"></link> -->
   <link name="imu">
     <collision>
@@ -388,4 +389,5 @@
     <dynamics damping="1.0" friction="1.0"/>
   </joint>
+<!--
   <joint type="fixed" name="camera_joint">
     <origin xyz="0.2 0 0" rpy="0 0 0"/>
@@ -393,10 +395,10 @@
     <parent link="chassis"/>
     <axis xyz="0 1 0" rpy="0 0 0"/>
-  </joint>
-  <joint name="camera_optical_joint" type="fixed">
+  </joint> -->
+  <!-- <joint name="camera_optical_joint" type="fixed">
     <origin xyz="0 0 0" rpy="-1.5707 0 -1.5707"/>
     <parent link="camera"/>
     <child link="camera_link_optical"/>
-  </joint>
+  </joint> -->
   <!--Lidar-->
   <xacro:arg name="gpu" default="false"/>
@@ -413,3 +415,5 @@
     <axis xyz="0 0 0" rpy="0 0 0"/>
   </joint>
+  <pan_tilt/>
+  <visible_camera/>
 </robot>

Commit message: Updated neck link and length

File: urdf/robot.xacro (robot description, xacro)
@@ -71,11 +71,11 @@
       <origin xyz="0 0 0" rpy=" 0 0 0"/>
       <geometry>
-        <cylinder length="0.55" radius="0.04"/>
-      </geometry>
-    </collision>
-    <visual name='chassis_visual'>
-      <origin xyz="0 0 0" rpy=" 0 0 0"/>
-      <geometry>
-        <cylinder length="0.55" radius="0.04"/>
+        <cylinder length="0.40" radius="0.04"/>
+      </geometry>
+    </collision>
+    <visual name='neck_visual'>
+      <origin xyz="0 0 0" rpy=" 0 0 0"/>
+      <geometry>
+        <cylinder length="0.40" radius="0.04"/>
       </geometry>
     </visual>
@@ -405,6 +405,6 @@
   <xacro:property name="gpu" value="$(arg gpu)" />
   <xacro:include filename="$(find robosense_description)/urdf/RS-16.urdf.xacro"/>
-  <RS-16 parent="chassis" name="rslidar" topic="/rslidar_points" hz="10" samples="150" gpu="${gpu}">
-    <origin xyz=".15 0 0.6" rpy="0 0 0" />
+  <RS-16 parent="neck" name="rslidar" topic="/rslidar_points" hz="10" samples="150" gpu="${gpu}">
+    <origin xyz="0 0 0.20" rpy="0 0 0" />
   </RS-16>
 <link name='scan'/>
