Commit message: Created auxiliar tf

File: urdf/visible_camera.xacro (robot description, xacro)
@@ -33,4 +33,10 @@
             <origin xyz="${visible_camera_x_distance} 0 ${visible_camera_z_distance}" rpy="0 0 0"/>
         </joint>
+        <link name="visible_camera_rotation_link"/>
+        <joint name="visible_camera_rotation_joint" type="fixed">
+            <parent link="visible_camera_link"/>
+            <child link="visible_camera_rotation_link"/>
+            <origin xyz="0 0 0" rpy="-1.57 0 -1.57"/>
+        </joint>
         <!-- camera -->
       <gazebo reference="visible_camera_link">
@@ -60,5 +66,5 @@
             <imageTopicName>image_raw</imageTopicName>
             <cameraInfoTopicName>camera_info</cameraInfoTopicName>
-            <frameName>visible_camera_link</frameName>
+            <frameName>visible_camera_rotation_link</frameName>
             <hackBaseline>0.07</hackBaseline>
             <distortionK1>0.0</distortionK1>
